File: SCHEMATIC/scheda PSE/AT24C256_EEPROM.kicad_sch (KiCad schematic)
At the start: 1 part

Commit message: sistemato tutto, e aggiunti i footprint da modificare
sistemato tutto, aggiunto e modificato i footprint.
Manca solo aggiungere i restanti footprint (praticamente solo dei componenti comuni)
Parts:
- removed U?: AT24C256, symbol altro:AT24C256
Changed lines of the file:
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@@
 (kicad_sch (version 20211123) (generator eeschema)
   (paper "A4")
-  (junction (at 130.81 92.71) (diameter 0) (color 0 0 0 0)
-  )
-  (junction (at 142.24 104.14) (diameter 0) (color 0 0 0 0)
-  )
-  (wire (pts (xy 130.81 88.9) (xy 130.81 92.71))
-    (stroke (width 0) (type default) (color 0 0 0 0))
-  )
-  (wire (pts (xy 142.24 104.14) (xy 142.24 105.41))
-    (stroke (width 0) (type default) (color 0 0 0 0))
-  )
-  (wire (pts (xy 142.24 102.87) (xy 142.24 104.14))
-    (stroke (width 0) (type default) (color 0 0 0 0))
-  )
-  (wire (pts (xy 133.35 88.9) (xy 130.81 88.9))
-    (stroke (width 0) (type default) (color 0 0 0 0))
-  )
-  (wire (pts (xy 130.81 92.71) (xy 133.35 92.71))
-    (stroke (width 0) (type default) (color 0 0 0 0))
-  )
-  (wire (pts (xy 154.94 83.82) (xy 158.75 83.82))
-    (stroke (width 0) (type default) (color 0 0 0 0))
-  )
-  (wire (pts (xy 151.13 88.9) (xy 154.94 88.9))
-    (stroke (width 0) (type default) (color 0 0 0 0))
-  )
-  (wire (pts (xy 142.24 81.28) (xy 142.24 83.82))
-    (stroke (width 0) (type default) (color 0 0 0 0))
-  )
-  (wire (pts (xy 151.13 92.71) (xy 156.21 92.71))
-    (stroke (width 0) (type default) (color 0 0 0 0))
-  )
-  (wire (pts (xy 130.81 104.14) (xy 142.24 104.14))
-    (stroke (width 0) (type default) (color 0 0 0 0))
-  )
-  (wire (pts (xy 130.81 92.71) (xy 130.81 104.14))
-    (stroke (width 0) (type default) (color 0 0 0 0))
-  )
-  (wire (pts (xy 151.13 96.52) (xy 156.21 96.52))
-    (stroke (width 0) (type default) (color 0 0 0 0))
-  )
-  (wire (pts (xy 158.75 83.82) (xy 158.75 85.09))
-    (stroke (width 0) (type default) (color 0 0 0 0))
-  )
-  (wire (pts (xy 154.94 88.9) (xy 154.94 83.82))
-    (stroke (width 0) (type default) (color 0 0 0 0))
-  )
-  (hierarchical_label "EEPROM_SCL" (shape input) (at 156.21 92.71 0)
-    (effects (font (size 1.27 1.27)) (justify left))
-  )
-  (hierarchical_label "EEPROM_SDA" (shape input) (at 156.21 96.52 0)
-    (effects (font (size 1.27 1.27)) (justify left))
-  )
-  (symbol (lib_id "altro:AT24C256") (at 142.24 92.71 0) (unit 1)
-    (in_bom yes) (on_board yes)
-    (property "Reference" "U?" (id 0) (at 146.05 81.28 0))
-    (property "Value" "AT24C256" (id 1) (at 148.59 83.82 0))
-    (property "Footprint" "" (id 2) (at 142.24 92.71 0)
-      (effects (font (size 1.27 1.27)) hide)
-    )
-    (property "Datasheet" "" (id 3) (at 142.24 92.71 0)
-      (effects (font (size 1.27 1.27)) hide)
-    )
-    (pin "1")
-    (pin "2")
-    (pin "3")
-    (pin "4")
-    (pin "5")
-    (pin "6")
-    (pin "7")
-    (pin "8")
-  )
-  (symbol (lib_id "power:+3.3V") (at 142.24 81.28 0) (unit 1)
-    (in_bom yes) (on_board yes) (fields_autoplaced)
-    (property "Reference" "#PWR?" (id 0) (at 142.24 85.09 0)
-      (effects (font (size 1.27 1.27)) hide)
-    )
-    (property "Value" "+3.3V" (id 1) (at 142.24 76.2 0))
-    (property "Footprint" "" (id 2) (at 142.24 81.28 0)
-      (effects (font (size 1.27 1.27)) hide)
-    )
-    (property "Datasheet" "" (id 3) (at 142.24 81.28 0)
-      (effects (font (size 1.27 1.27)) hide)
-    )
-    (pin "1")
-  )
-  (symbol (lib_id "power:GND") (at 142.24 105.41 0) (unit 1)
-    (in_bom yes) (on_board yes) (fields_autoplaced)
-    (property "Reference" "#PWR?" (id 0) (at 142.24 111.76 0)
-      (effects (font (size 1.27 1.27)) hide)
-    )
-    (property "Value" "GND" (id 1) (at 142.24 110.49 0))
-    (property "Footprint" "" (id 2) (at 142.24 105.41 0)
-      (effects (font (size 1.27 1.27)) hide)
-    )
-    (property "Datasheet" "" (id 3) (at 142.24 105.41 0)
-      (effects (font (size 1.27 1.27)) hide)
-    )
-    (pin "1")
-  )
-  (symbol (lib_id "power:GND") (at 158.75 85.09 0) (unit 1)
-    (in_bom yes) (on_board yes)
-    (property "Reference" "#PWR?" (id 0) (at 158.75 91.44 0)
-      (effects (font (size 1.27 1.27)) hide)
-    )
-    (property "Value" "GND" (id 1) (at 161.29 88.9 0))
-    (property "Footprint" "" (id 2) (at 158.75 85.09 0)
-      (effects (font (size 1.27 1.27)) hide)
-    )
-    (property "Datasheet" "" (id 3) (at 158.75 85.09 0)
-      (effects (font (size 1.27 1.27)) hide)
-    )
-    (pin "1")
-  )
 )
