File: SCHEMATIC/scheda PSE/sensori.kicad_sch (KiCad schematic)
At the start: 17 parts, among them J5 I2C_3V3, J6 UART0_3V3, Q3 IRLML9301, U7 SAM-M8Q, U8 MMA8451Q, U9 TC1047A

Commit message: iniziato lo broglio. Prima di continuare modificare pin schema
iniziato lo sbroglio della scheda, prima di continuare bisogna sistemare i pin che siano concordi con quelli degli altro (ovvero sistemarli come da tabella su telegram)
Connections:
- net +3.3V is gone; now on net +3V3: J5.1 (Pin_1), J6.1 (Pin_1)
- net +3V3: no longer C43.1, U9.1 (Vdd)
- new net +3.3VA: C43.1, U9.1 (Vdd)
Changed lines of the file:
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@@
   (symbol (lib_id "power:GND") (at 132.715 67.31 0) (unit 1)
     (in_bom yes) (on_board yes) (fields_autoplaced)
-    (property "Reference" "#PWR080" (id 0) (at 132.715 73.66 0)
+    (property "Reference" "#PWR079" (id 0) (at 132.715 73.66 0)
       (effects (font (size 1.27 1.27)) hide)
     )
@@
   (symbol (lib_id "power:GND") (at 165.735 67.31 0) (unit 1)
     (in_bom yes) (on_board yes) (fields_autoplaced)
-    (property "Reference" "#PWR082" (id 0) (at 165.735 73.66 0)
+    (property "Reference" "#PWR081" (id 0) (at 165.735 73.66 0)
       (effects (font (size 1.27 1.27)) hide)
     )
@@
   (symbol (lib_id "power:GND") (at 106.045 108.585 0) (unit 1)
     (in_bom yes) (on_board yes) (fields_autoplaced)
-    (property "Reference" "#PWR077" (id 0) (at 106.045 114.935 0)
+    (property "Reference" "#PWR076" (id 0) (at 106.045 114.935 0)
       (effects (font (size 1.27 1.27)) hide)
     )
@@
   (symbol (lib_id "power:GND") (at 92.075 62.865 0) (unit 1)
     (in_bom yes) (on_board yes) (fields_autoplaced)
-    (property "Reference" "#PWR075" (id 0) (at 92.075 69.215 0)
+    (property "Reference" "#PWR074" (id 0) (at 92.075 69.215 0)
       (effects (font (size 1.27 1.27)) hide)
     )
@@
     (pin "1")
   )
-  (symbol (lib_id "power:+3.3V") (at 167.64 94.615 0) (unit 1)
-    (in_bom yes) (on_board yes) (fields_autoplaced)
-    (property "Reference" "#PWR083" (id 0) (at 167.64 98.425 0)
-      (effects (font (size 1.27 1.27)) hide)
-    )
-    (property "Value" "+3.3V" (id 1) (at 167.64 91.0392 0))
-    (property "Footprint" "" (id 2) (at 167.64 94.615 0)
-      (effects (font (size 1.27 1.27)) hide)
-    )
-    (property "Datasheet" "" (id 3) (at 167.64 94.615 0)
-      (effects (font (size 1.27 1.27)) hide)
-    )
-    (pin "1")
-  )
   (symbol (lib_id "power:GNDA") (at 190.5 56.515 0) (unit 1)
     (in_bom yes) (on_board yes)
-    (property "Reference" "#PWR085" (id 0) (at 190.5 62.865 0)
+    (property "Reference" "#PWR084" (id 0) (at 190.5 62.865 0)
       (effects (font (size 1.27 1.27)) hide)
     )
@@
   (symbol (lib_id "power:GND") (at 201.93 104.775 0) (unit 1)
     (in_bom yes) (on_board yes) (fields_autoplaced)
-    (property "Reference" "#PWR087" (id 0) (at 201.93 111.125 0)
+    (property "Reference" "#PWR086" (id 0) (at 201.93 111.125 0)
       (effects (font (size 1.27 1.27)) hide)
     )
@@
   (symbol (lib_id "power:GND") (at 113.665 67.31 0) (unit 1)
     (in_bom yes) (on_board yes) (fields_autoplaced)
-    (property "Reference" "#PWR078" (id 0) (at 113.665 73.66 0)
+    (property "Reference" "#PWR077" (id 0) (at 113.665 73.66 0)
       (effects (font (size 1.27 1.27)) hide)
     )
@@
   (symbol (lib_id "power:GNDA") (at 229.87 73.66 0) (unit 1)
     (in_bom yes) (on_board yes)
-    (property "Reference" "#PWR090" (id 0) (at 229.87 80.01 0)
+    (property "Reference" "#PWR089" (id 0) (at 229.87 80.01 0)
       (effects (font (size 1.27 1.27)) hide)
     )
@@
     (pin "1")
   )
-  (symbol (lib_id "power:+3.3V") (at 201.93 93.98 0) (unit 1)
-    (in_bom yes) (on_board yes) (fields_autoplaced)
-    (property "Reference" "#PWR086" (id 0) (at 201.93 97.79 0)
-      (effects (font (size 1.27 1.27)) hide)
-    )
-    (property "Value" "+3.3V" (id 1) (at 201.93 90.4042 0))
-    (property "Footprint" "" (id 2) (at 201.93 93.98 0)
-      (effects (font (size 1.27 1.27)) hide)
-    )
-    (property "Datasheet" "" (id 3) (at 201.93 93.98 0)
+  (symbol (lib_id "power:+3V3") (at 167.64 94.615 0) (unit 1)
+    (in_bom yes) (on_board yes)
+    (property "Reference" "#PWR082" (id 0) (at 167.64 98.425 0)
+      (effects (font (size 1.27 1.27)) hide)
+    )
+    (property "Value" "+3V3" (id 1) (at 167.005 90.805 0))
+    (property "Footprint" "" (id 2) (at 167.64 94.615 0)
+      (effects (font (size 1.27 1.27)) hide)
+    )
+    (property "Datasheet" "" (id 3) (at 167.64 94.615 0)
       (effects (font (size 1.27 1.27)) hide)
     )
@@
   (symbol (lib_id "power:GND") (at 167.64 105.41 0) (unit 1)
     (in_bom yes) (on_board yes) (fields_autoplaced)
-    (property "Reference" "#PWR084" (id 0) (at 167.64 111.76 0)
+    (property "Reference" "#PWR083" (id 0) (at 167.64 111.76 0)
       (effects (font (size 1.27 1.27)) hide)
     )
@@
     )
     (property "Datasheet" "" (id 3) (at 167.64 105.41 0)
+      (effects (font (size 1.27 1.27)) hide)
+    )
+    (pin "1")
+  )
+  (symbol (lib_id "power:+3V3") (at 201.93 93.98 0) (unit 1)
+    (in_bom yes) (on_board yes)
+    (property "Reference" "#PWR085" (id 0) (at 201.93 97.79 0)
+      (effects (font (size 1.27 1.27)) hide)
+    )
+    (property "Value" "+3V3" (id 1) (at 201.295 90.17 0))
+    (property "Footprint" "" (id 2) (at 201.93 93.98 0)
+      (effects (font (size 1.27 1.27)) hide)
+    )
+    (property "Datasheet" "" (id 3) (at 201.93 93.98 0)
       (effects (font (size 1.27 1.27)) hide)
     )
@@
     (pin "3")
   )
+  (symbol (lib_id "power:+3.3VA") (at 203.835 43.18 0) (unit 1)
+    (in_bom yes) (on_board yes) (fields_autoplaced)
+    (property "Reference" "#PWR087" (id 0) (at 203.835 46.99 0)
+      (effects (font (size 1.27 1.27)) hide)
+    )
+    (property "Value" "+3.3VA" (id 1) (at 203.835 39.6042 0))
+    (property "Footprint" "" (id 2) (at 203.835 43.18 0)
+      (effects (font (size 1.27 1.27)) hide)
+    )
+    (property "Datasheet" "" (id 3) (at 203.835 43.18 0)
+      (effects (font (size 1.27 1.27)) hide)
+    )
+    (pin "1")
+  )
   (symbol (lib_id "power:+3V3") (at 65.405 95.885 0) (unit 1)
     (in_bom yes) (on_board yes) (fields_autoplaced)
-    (property "Reference" "#PWR071" (id 0) (at 65.405 99.695 0)
+    (property "Reference" "#PWR070" (id 0) (at 65.405 99.695 0)
       (effects (font (size 1.27 1.27)) hide)
     )
@@
   (symbol (lib_id "power:+3V3") (at 137.795 29.21 0) (unit 1)
     (in_bom yes) (on_board yes)
-    (property "Reference" "#PWR081" (id 0) (at 137.795 33.02 0)
+    (property "Reference" "#PWR080" (id 0) (at 137.795 33.02 0)
       (effects (font (size 1.27 1.27)) hide)
     )
@@
   (symbol (lib_id "power:+3V3") (at 92.075 41.275 0) (unit 1)
     (in_bom yes) (on_board yes)
-    (property "Reference" "#PWR074" (id 0) (at 92.075 45.085 0)
+    (property "Reference" "#PWR073" (id 0) (at 92.075 45.085 0)
       (effects (font (size 1.27 1.27)) hide)
     )
@@
   (symbol (lib_id "power:GND") (at 117.475 153.035 0) (unit 1)
     (in_bom yes) (on_board yes) (fields_autoplaced)
-    (property "Reference" "#PWR079" (id 0) (at 117.475 159.385 0)
+    (property "Reference" "#PWR078" (id 0) (at 117.475 159.385 0)
       (effects (font (size 1.27 1.27)) hide)
     )
@@
   (symbol (lib_id "power:GND") (at 95.885 108.585 0) (unit 1)
     (in_bom yes) (on_board yes) (fields_autoplaced)
-    (property "Reference" "#PWR076" (id 0) (at 95.885 114.935 0)
+    (property "Reference" "#PWR075" (id 0) (at 95.885 114.935 0)
       (effects (font (size 1.27 1.27)) hide)
     )
@@
   (symbol (lib_id "power:+3V3") (at 85.09 41.275 0) (unit 1)
     (in_bom yes) (on_board yes)
-    (property "Reference" "#PWR073" (id 0) (at 85.09 45.085 0)
+    (property "Reference" "#PWR072" (id 0) (at 85.09 45.085 0)
       (effects (font (size 1.27 1.27)) hide)
     )
@@
     (pin "1")
   )
-  (symbol (lib_id "power:+3V3") (at 203.835 43.18 0) (unit 1)
-    (in_bom yes) (on_board yes)
-    (property "Reference" "#PWR088" (id 0) (at 203.835 46.99 0)
-      (effects (font (size 1.27 1.27)) hide)
-    )
-    (property "Value" "+3V3" (id 1) (at 203.835 39.37 0))
-    (property "Footprint" "" (id 2) (at 203.835 43.18 0)
-      (effects (font (size 1.27 1.27)) hide)
-    )
-    (property "Datasheet" "" (id 3) (at 203.835 43.18 0)
-      (effects (font (size 1.27 1.27)) hide)
-    )
-    (pin "1")
-  )
   (symbol (lib_id "Device:R") (at 85.09 59.69 0) (unit 1)
     (in_bom yes) (on_board yes)
@@
   (symbol (lib_id "power:GNDA") (at 203.835 73.66 0) (unit 1)
     (in_bom yes) (on_board yes)
-    (property "Reference" "#PWR089" (id 0) (at 203.835 80.01 0)
+    (property "Reference" "#PWR088" (id 0) (at 203.835 80.01 0)
       (effects (font (size 1.27 1.27)) hide)
     )
@@
   (symbol (lib_id "power:+3V3") (at 78.105 41.275 0) (unit 1)
     (in_bom yes) (on_board yes)
-    (property "Reference" "#PWR072" (id 0) (at 78.105 45.085 0)
-      (effects (font (size 1.27 1.27)) hide)
-    )
+    (property "Reference" "#PWR071" (id 0) (at 78.105 45.085 0)
+      (effects (font (size 1.27 1.27)) hide)
+    )

Commit message: sistemato buzzer, e continuato lo sbroglio
sistemato il buzzer con un altro footprint e ho continuato lo sbroglio.
Teoricamente manca solo collegare i collegamenti tra le gpio del rp2040 e il resto dei componenti
Parts:
- renumbered R22 to R21, R23 to R22, R24 to R23, R25 to R24
Changed lines of the file:
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@@
   (symbol (lib_id "Device:R") (at 78.105 59.69 0) (unit 1)
     (in_bom yes) (on_board yes)
-    (property "Reference" "R23" (id 0) (at 79.375 58.42 0)
+    (property "Reference" "R22" (id 0) (at 79.375 58.42 0)
       (effects (font (size 1.27 1.27)) (justify left))
     )
@@
   (symbol (lib_id "Device:R") (at 221.615 62.23 90) (unit 1)
     (in_bom yes) (on_board yes) (fields_autoplaced)
-    (property "Reference" "R25" (id 0) (at 221.615 57.5142 90))
+    (property "Reference" "R24" (id 0) (at 221.615 57.5142 90))
     (property "Value" "470" (id 1) (at 221.615 60.0511 90))
     (property "Footprint" "Resistor_SMD:R_0603_1608Metric" (id 2) (at 221.615 64.008 90)
@@
   (symbol (lib_id "Device:R") (at 73.025 106.045 90) (unit 1)
     (in_bom yes) (on_board yes) (fields_autoplaced)
-    (property "Reference" "R22" (id 0) (at 73.025 101.3292 90))
+    (property "Reference" "R21" (id 0) (at 73.025 101.3292 90))
     (property "Value" "10k" (id 1) (at 73.025 103.8661 90))
     (property "Footprint" "Resistor_SMD:R_0603_1608Metric" (id 2) (at 73.025 107.823 90)
@@
   (symbol (lib_id "Device:R") (at 85.09 59.69 0) (unit 1)
     (in_bom yes) (on_board yes)
-    (property "Reference" "R24" (id 0) (at 86.36 58.42 0)
-      (effects (font (size 1.27 1.27)) (justify left))
-    )
+    (property "Reference" "R23" (id 0) (at 86.36 58.42 0)
+      (effects (font (size 1.27 1.27)) (justify left))
+    )

Commit message: modificato pin 2,3,14,15,16,17,18,27,28,29,30,31,32
Connections:
- net SAM_RST: now reaches U7.18 (~{RESET})
- net PPS_SAM: now reaches U7.7 (TIMEPULSE)
- no-connect marks 11 -> 9
Changed lines of the file:
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@@
   )
   (no_connect (at 132.715 34.29))
-  (no_connect (at 104.775 135.255))
   (no_connect (at 104.775 137.795))
   (no_connect (at 127.635 34.29))
@@
   (no_connect (at 149.225 43.18))
   (no_connect (at 104.775 132.715))
-  (no_connect (at 104.775 140.335))
   (no_connect (at 130.175 137.795))
   (no_connect (at 137.795 66.04))
@@
     (stroke (width 0) (type default) (color 0 0 0 0))
   )
+  (wire (pts (xy 95.25 135.255) (xy 104.775 135.255))
+    (stroke (width 0) (type default) (color 0 0 0 0))
+  )
   (polyline (pts (xy 61.595 86.36) (xy 61.595 161.29))
     (stroke (width 0) (type default) (color 0 0 0 0))
@@
   )
   (wire (pts (xy 149.225 46.99) (xy 165.735 46.99))
+    (stroke (width 0) (type default) (color 0 0 0 0))
+  )
+  (wire (pts (xy 95.25 140.335) (xy 104.775 140.335))
     (stroke (width 0) (type default) (color 0 0 0 0))
   )
@@
     (effects (font (size 1.27 1.27)) (justify left))
   )
+  (hierarchical_label "PPS_SAM" (shape output) (at 95.25 135.255 180)
+    (effects (font (size 1.27 1.27)) (justify right))
+  )
   (hierarchical_label "TX_SAM" (shape output) (at 136.525 132.715 0)
     (effects (font (size 1.27 1.27)) (justify left))
@@
     (effects (font (size 1.27 1.27)) (justify left))
   )
+  (hierarchical_label "SAM_RST" (shape input) (at 95.25 140.335 180)
+    (effects (font (size 1.27 1.27)) (justify right))
+  )
   (symbol (lib_id "Connector_Generic:Conn_01x04") (at 208.915 97.79 0) (unit 1)

Commit message: finito lo sbroglio (magari da ricontrollare)
finito lo sbroglio, controllato già io ma meglio ridare una controllata.
Da sistemare tutta la serigrafia
Connections:
- net GND: no longer U8.7 (SA0)
- net PPS_SAM renamed SAM_PPS
- new net ACC_SA0: U8.7 (SA0)
Changed lines of the file:
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@@
+    (stroke (width 0) (type default) (color 0 0 0 0))
+  )
+  (wire (pts (xy 132.715 66.04) (xy 132.715 68.58))
     (stroke (width 0) (type default) (color 0 0 0 0))
   )
@@
   )
   (polyline (pts (xy 175.895 80.01) (xy 61.595 80.01))
-    (stroke (width 0) (type default) (color 0 0 0 0))
-  )
-  (wire (pts (xy 132.715 66.04) (xy 132.715 67.31))
     (stroke (width 0) (type default) (color 0 0 0 0))
   )
@@
     (effects (font (size 1.27 1.27)) (justify right))
   )
+  (hierarchical_label "ACC_SA0" (shape input) (at 132.715 68.58 270)
+    (effects (font (size 1.27 1.27)) (justify right))
+  )
   (hierarchical_label "EXT_UART0_TX" (shape output) (at 200.025 97.79 180)
     (effects (font (size 1.27 1.27)) (justify right))
@@
     (effects (font (size 1.27 1.27)) (justify left))
   )
-  (hierarchical_label "PPS_SAM" (shape output) (at 95.25 135.255 180)
+  (hierarchical_label "SAM_PPS" (shape output) (at 95.25 135.255 180)
     (effects (font (size 1.27 1.27)) (justify right))
   )
@@
     (pin "4")
   )
-  (symbol (lib_id "power:GND") (at 132.715 67.31 0) (unit 1)
-    (in_bom yes) (on_board yes) (fields_autoplaced)
-    (property "Reference" "#PWR079" (id 0) (at 132.715 73.66 0)
-      (effects (font (size 1.27 1.27)) hide)
-    )
-    (property "Value" "GND" (id 1) (at 132.715 71.7534 0))
-    (property "Footprint" "" (id 2) (at 132.715 67.31 0)
-      (effects (font (size 1.27 1.27)) hide)
-    )
-    (property "Datasheet" "" (id 3) (at 132.715 67.31 0)
-      (effects (font (size 1.27 1.27)) hide)
-    )
-    (pin "1")
-  )
   (symbol (lib_id "Device:C") (at 103.505 51.435 0) (unit 1)
