File: SCHEMATIC/scheda PSE/alimentazione.kicad_sch (KiCad schematic)
At the start: 39 parts, among them J2 Vin, J3 USB_B_Mini, J4 Vout 5V, SW7 Power_button, U5 TPS563201, U6 XC6705A331MR-G

Commit message: Posizionati tutti i componenti
Posizionati tutti i componenti sulla scheda
Parts:
- added TP2: 5V, TestPoint:TestPoint_THTPad_D1.5mm_Drill0.7mm, symbol Connector:TestPoint
- TP1: footprint TestPoint:TestPoint_Loop_D2.50mm_Drill1.0mm_LowProfile -> TestPoint:TestPoint_THTPad_D1.5mm_Drill0.7mm
- TP3: renamed from TP2; footprint TestPoint:TestPoint_Loop_D2.50mm_Drill1.0mm_LowProfile -> TestPoint:TestPoint_THTPad_D1.5mm_Drill0.7mm
- TP4: renamed from TP3; footprint TestPoint:TestPoint_Loop_D2.50mm_Drill1.0mm_LowProfile -> TestPoint:TestPoint_THTPad_D1.5mm_Drill0.7mm
Connections:
- net +5V: now also TP2.1
Changed lines of the file:
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@@
   (junction (at 73.66 95.885) (diameter 0) (color 0 0 0 0)
+  )
+  (junction (at 154.94 54.61) (diameter 0) (color 0 0 0 0)
   )
   (junction (at 216.535 73.025) (diameter 0) (color 0 0 0 0)
@@
     (stroke (width 0) (type default) (color 0 0 0 0))
   )
+  (wire (pts (xy 154.94 54.61) (xy 160.02 54.61))
+    (stroke (width 0) (type default) (color 0 0 0 0))
+  )
   (wire (pts (xy 160.02 59.69) (xy 160.02 54.61))
     (stroke (width 0) (type default) (color 0 0 0 0))
@@
     (stroke (width 0) (type default) (color 0 0 0 0))
   )
-  (wire (pts (xy 148.59 54.61) (xy 160.02 54.61))
+  (wire (pts (xy 148.59 54.61) (xy 154.94 54.61))
     (stroke (width 0) (type default) (color 0 0 0 0))
   )
@@
       (effects (font (size 1.27 1.27)) (justify left))
     )
-    (property "Footprint" "TestPoint:TestPoint_Loop_D2.50mm_Drill1.0mm_LowProfile" (id 2) (at 78.74 50.8 0)
+    (property "Footprint" "TestPoint:TestPoint_THTPad_D1.5mm_Drill0.7mm" (id 2) (at 78.74 50.8 0)
       (effects (font (size 1.27 1.27)) hide)
     )
@@
   (symbol (lib_id "Connector:TestPoint") (at 196.85 53.975 0) (unit 1)
     (in_bom yes) (on_board yes)
-    (property "Reference" "TP2" (id 0) (at 198.12 50.8 0)
+    (property "Reference" "TP3" (id 0) (at 198.12 50.8 0)
       (effects (font (size 1.27 1.27)) (justify left))
     )
@@
       (effects (font (size 1.27 1.27)) (justify left))
     )
-    (property "Footprint" "TestPoint:TestPoint_Loop_D2.50mm_Drill1.0mm_LowProfile" (id 2) (at 201.93 53.975 0)
+    (property "Footprint" "TestPoint:TestPoint_THTPad_D1.5mm_Drill0.7mm" (id 2) (at 201.93 53.975 0)
       (effects (font (size 1.27 1.27)) hide)
     )
@@
     (pin "1")
   )
+  (symbol (lib_id "Connector:TestPoint") (at 154.94 54.61 0) (mirror y) (unit 1)
+    (in_bom yes) (on_board yes)
+    (property "Reference" "TP2" (id 0) (at 153.67 50.8 0)
+      (effects (font (size 1.27 1.27)) (justify left))
+    )
+    (property "Value" "5V" (id 1) (at 153.67 53.3369 0)
+      (effects (font (size 1.27 1.27)) (justify left))
+    )
+    (property "Footprint" "TestPoint:TestPoint_THTPad_D1.5mm_Drill0.7mm" (id 2) (at 149.86 54.61 0)
+      (effects (font (size 1.27 1.27)) hide)
+    )
+    (property "Datasheet" "~" (id 3) (at 149.86 54.61 0)
+      (effects (font (size 1.27 1.27)) hide)
+    )
+    (pin "1")
+  )
   (symbol (lib_id "Device:C_Small") (at 163.83 99.06 0) (unit 1)
     (in_bom yes) (on_board yes) (fields_autoplaced)
@@
   (symbol (lib_id "Connector:TestPoint") (at 226.06 64.135 270) (unit 1)
     (in_bom yes) (on_board yes)
-    (property "Reference" "TP3" (id 0) (at 231.14 66.675 90)
+    (property "Reference" "TP4" (id 0) (at 231.14 66.675 90)
       (effects (font (size 1.27 1.27)) (justify right))
     )
@@
       (effects (font (size 1.27 1.27)) (justify right))
     )
-    (property "Footprint" "TestPoint:TestPoint_Loop_D2.50mm_Drill1.0mm_LowProfile" (id 2) (at 226.06 69.215 0)
-      (effects (font (size 1.27 1.27)) hide)
-    )
+    (property "Footprint" "TestPoint:TestPoint_THTPad_D1.5mm_Drill0.7mm" (id 2) (at 226.06 69.215 0)
+      (effects (font (size 1.27 1.27)) hide)
+    )

Commit message: iniziato lo broglio. Prima di continuare modificare pin schema
iniziato lo sbroglio della scheda, prima di continuare bisogna sistemare i pin che siano concordi con quelli degli altro (ovvero sistemarli come da tabella su telegram)
Connections:
- net D-: now reaches J3.2 (D-), R15.2
- net D+: now reaches J3.3 (D+), R14.1
- net USB_DM renamed USB_DN
Changed lines of the file:
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@@
+    (effects (font (size 1.27 1.27)) (justify left bottom))
+  )
+  (label "D+" (at 84.455 62.865 0)
+    (effects (font (size 1.27 1.27)) (justify left bottom))
+  )
+  (label "D-" (at 84.455 65.405 0)
     (effects (font (size 1.27 1.27)) (justify left bottom))
   )
@@
     (effects (font (size 1.27 1.27)) (justify right))
   )
-  (hierarchical_label "USB_DM" (shape bidirectional) (at 101.6 65.405 0)
+  (hierarchical_label "USB_DN" (shape bidirectional) (at 101.6 65.405 0)
     (effects (font (size 1.27 1.27)) (justify left))
   )
@@
   (symbol (lib_id "power:+5V") (at 249.555 95.25 0) (unit 1)
     (in_bom yes) (on_board yes) (fields_autoplaced)
-    (property "Reference" "#PWR069" (id 0) (at 249.555 99.06 0)
+    (property "Reference" "#PWR068" (id 0) (at 249.555 99.06 0)
       (effects (font (size 1.27 1.27)) hide)
     )
@@
   (symbol (lib_id "power:GND") (at 186.69 67.31 0) (unit 1)
     (in_bom yes) (on_board yes) (fields_autoplaced)
-    (property "Reference" "#PWR060" (id 0) (at 186.69 73.66 0)
+    (property "Reference" "#PWR059" (id 0) (at 186.69 73.66 0)
       (effects (font (size 1.27 1.27)) hide)
     )
@@
   (symbol (lib_id "power:GND") (at 48.26 106.68 0) (unit 1)
     (in_bom yes) (on_board yes) (fields_autoplaced)
-    (property "Reference" "#PWR046" (id 0) (at 48.26 113.03 0)
+    (property "Reference" "#PWR045" (id 0) (at 48.26 113.03 0)
       (effects (font (size 1.27 1.27)) hide)
     )
@@
   (symbol (lib_id "power:GND") (at 73.66 108.585 0) (unit 1)
     (in_bom yes) (on_board yes) (fields_autoplaced)
-    (property "Reference" "#PWR049" (id 0) (at 73.66 114.935 0)
+    (property "Reference" "#PWR048" (id 0) (at 73.66 114.935 0)
       (effects (font (size 1.27 1.27)) hide)
     )
@@
   (symbol (lib_id "power:GND") (at 269.875 100.33 0) (unit 1)
     (in_bom yes) (on_board yes) (fields_autoplaced)
-    (property "Reference" "#PWR070" (id 0) (at 269.875 106.68 0)
+    (property "Reference" "#PWR069" (id 0) (at 269.875 106.68 0)
       (effects (font (size 1.27 1.27)) hide)
     )
@@
   (symbol (lib_id "power:GND") (at 177.165 113.665 0) (unit 1)
     (in_bom yes) (on_board yes) (fields_autoplaced)
-    (property "Reference" "#PWR059" (id 0) (at 177.165 120.015 0)
+    (property "Reference" "#PWR058" (id 0) (at 177.165 120.015 0)
       (effects (font (size 1.27 1.27)) hide)
     )
@@
   (symbol (lib_id "power:GND") (at 92.71 108.585 0) (unit 1)
     (in_bom yes) (on_board yes) (fields_autoplaced)
-    (property "Reference" "#PWR052" (id 0) (at 92.71 114.935 0)
+    (property "Reference" "#PWR051" (id 0) (at 92.71 114.935 0)
       (effects (font (size 1.27 1.27)) hide)
     )
@@
   (symbol (lib_id "power:+3V3") (at 189.865 53.34 0) (unit 1)
     (in_bom yes) (on_board yes) (fields_autoplaced)
-    (property "Reference" "#PWR061" (id 0) (at 189.865 57.15 0)
+    (property "Reference" "#PWR060" (id 0) (at 189.865 57.15 0)
       (effects (font (size 1.27 1.27)) hide)
     )
@@
   (symbol (lib_id "power:GND") (at 217.17 108.585 0) (unit 1)
     (in_bom yes) (on_board yes) (fields_autoplaced)
-    (property "Reference" "#PWR064" (id 0) (at 217.17 114.935 0)
+    (property "Reference" "#PWR063" (id 0) (at 217.17 114.935 0)
       (effects (font (size 1.27 1.27)) hide)
     )
@@
   (symbol (lib_id "power:GND") (at 31.75 100.965 0) (unit 1)
     (in_bom yes) (on_board yes) (fields_autoplaced)
-    (property "Reference" "#PWR045" (id 0) (at 31.75 107.315 0)
+    (property "Reference" "#PWR044" (id 0) (at 31.75 107.315 0)
       (effects (font (size 1.27 1.27)) hide)
     )
@@
   (symbol (lib_id "power:GND") (at 83.185 108.585 0) (unit 1)
     (in_bom yes) (on_board yes) (fields_autoplaced)
-    (property "Reference" "#PWR051" (id 0) (at 83.185 114.935 0)
+    (property "Reference" "#PWR050" (id 0) (at 83.185 114.935 0)
       (effects (font (size 1.27 1.27)) hide)
     )
@@
   (symbol (lib_id "power:GND") (at 141.605 113.665 0) (unit 1)
     (in_bom yes) (on_board yes) (fields_autoplaced)
-    (property "Reference" "#PWR055" (id 0) (at 141.605 120.015 0)
+    (property "Reference" "#PWR054" (id 0) (at 141.605 120.015 0)
       (effects (font (size 1.27 1.27)) hide)
     )
@@
   (symbol (lib_id "power:+5V") (at 145.415 53.34 0) (unit 1)
     (in_bom yes) (on_board yes) (fields_autoplaced)
-    (property "Reference" "#PWR056" (id 0) (at 145.415 57.15 0)
+    (property "Reference" "#PWR055" (id 0) (at 145.415 57.15 0)
       (effects (font (size 1.27 1.27)) hide)
     )
@@
   (symbol (lib_id "power:GND") (at 148.59 67.31 0) (unit 1)
     (in_bom yes) (on_board yes) (fields_autoplaced)
-    (property "Reference" "#PWR057" (id 0) (at 148.59 73.66 0)
+    (property "Reference" "#PWR056" (id 0) (at 148.59 73.66 0)
       (effects (font (size 1.27 1.27)) hide)
     )
@@
   (symbol (lib_id "power:+12V") (at 81.28 129.54 0) (unit 1)
     (in_bom yes) (on_board yes) (fields_autoplaced)
-    (property "Reference" "#PWR050" (id 0) (at 81.28 133.35 0)
+    (property "Reference" "#PWR049" (id 0) (at 81.28 133.35 0)
       (effects (font (size 1.27 1.27)) hide)
     )
@@
   (symbol (lib_id "power:GND") (at 119.38 111.125 0) (unit 1)
     (in_bom yes) (on_board yes) (fields_autoplaced)
-    (property "Reference" "#PWR053" (id 0) (at 119.38 117.475 0)
+    (property "Reference" "#PWR052" (id 0) (at 119.38 117.475 0)
       (effects (font (size 1.27 1.27)) hide)
     )
@@
   (symbol (lib_id "power:+12V") (at 73.66 94.615 0) (unit 1)
     (in_bom yes) (on_board yes) (fields_autoplaced)
-    (property "Reference" "#PWR048" (id 0) (at 73.66 98.425 0)
+    (property "Reference" "#PWR047" (id 0) (at 73.66 98.425 0)
       (effects (font (size 1.27 1.27)) hide)
     )
@@
   (symbol (lib_id "power:+3.3VA") (at 225.425 62.23 0) (unit 1)
     (in_bom yes) (on_board yes) (fields_autoplaced)
-    (property "Reference" "#PWR065" (id 0) (at 225.425 66.04 0)
+    (property "Reference" "#PWR064" (id 0) (at 225.425 66.04 0)
       (effects (font (size 1.27 1.27)) hide)
     )
@@
   (symbol (lib_id "power:GND") (at 196.85 73.66 0) (unit 1)
     (in_bom yes) (on_board yes) (fields_autoplaced)
-    (property "Reference" "#PWR062" (id 0) (at 196.85 80.01 0)
+    (property "Reference" "#PWR061" (id 0) (at 196.85 80.01 0)
       (effects (font (size 1.27 1.27)) hide)
     )
@@
   (symbol (lib_id "power:GND") (at 247.015 114.3 0) (unit 1)
     (in_bom yes) (on_board yes) (fields_autoplaced)
-    (property "Reference" "#PWR068" (id 0) (at 247.015 120.65 0)
+    (property "Reference" "#PWR067" (id 0) (at 247.015 120.65 0)
       (effects (font (size 1.27 1.27)) hide)
     )
@@
   (symbol (lib_id "power:+5V") (at 133.35 52.705 0) (unit 1)
     (in_bom yes) (on_board yes) (fields_autoplaced)
-    (property "Reference" "#PWR054" (id 0) (at 133.35 56.515 0)
+    (property "Reference" "#PWR053" (id 0) (at 133.35 56.515 0)
       (effects (font (size 1.27 1.27)) hide)
     )
@@
   (symbol (lib_id "power:GND") (at 236.855 108.585 0) (unit 1)
     (in_bom yes) (on_board yes) (fields_autoplaced)
-    (property "Reference" "#PWR067" (id 0) (at 236.855 114.935 0)
+    (property "Reference" "#PWR066" (id 0) (at 236.855 114.935 0)
       (effects (font (size 1.27 1.27)) hide)
     )
@@
   (symbol (lib_id "power:GND") (at 72.39 74.93 0) (unit 1)
     (in_bom yes) (on_board yes) (fields_autoplaced)
-    (property "Reference" "#PWR047" (id 0) (at 72.39 81.28 0)
+    (property "Reference" "#PWR046" (id 0) (at 72.39 81.28 0)
       (effects (font (size 1.27 1.27)) hide)
     )
@@
   (symbol (lib_id "power:GND") (at 171.45 67.31 0) (unit 1)
     (in_bom yes) (on_board yes) (fields_autoplaced)
-    (property "Reference" "#PWR058" (id 0) (at 171.45 73.66 0)
+    (property "Reference" "#PWR057" (id 0) (at 171.45 73.66 0)
       (effects (font (size 1.27 1.27)) hide)
     )
@@
   (symbol (lib_id "power:GNDA") (at 216.535 73.66 0) (unit 1)
     (in_bom yes) (on_board yes) (fields_autoplaced)
-    (property "Reference" "#PWR063" (id 0) (at 216.535 80.01 0)
+    (property "Reference" "#PWR062" (id 0) (at 216.535 80.01 0)
       (effects (font (size 1.27 1.27)) hide)
     )
@@
   (symbol (lib_id "power:GND") (at 227.33 108.585 0) (unit 1)
     (in_bom yes) (on_board yes) (fields_autoplaced)
-    (property "Reference" "#PWR066" (id 0) (at 227.33 114.935 0)
-      (effects (font (size 1.27 1.27)) hide)
-    )
+    (property "Reference" "#PWR065" (id 0) (at 227.33 114.935 0)
+      (effects (font (size 1.27 1.27)) hide)
+    )

Commit message: sistemato buzzer, e continuato lo sbroglio
sistemato il buzzer con un altro footprint e ho continuato lo sbroglio.
Teoricamente manca solo collegare i collegamenti tra le gpio del rp2040 e il resto dei componenti
Parts:
- renumbered D10 to D11, D11 to D12, D12 to D13, D13 to D14, D14 to D15, D15 to D16, D16 to D17, D17 to D18, R14 to R13, R15 to R14, R16 to R15, R17 to R16, R18 to R17, R19 to R18, R20 to R19, R21 to R20
Changed lines of the file:
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@@
   (symbol (lib_id "Device:D_Schottky") (at 258.445 95.885 180) (unit 1)
     (in_bom yes) (on_board yes)
-    (property "Reference" "D17" (id 0) (at 258.445 92.71 0))
+    (property "Reference" "D18" (id 0) (at 258.445 92.71 0))
     (property "Value" "RBR1VWM30ATFTR" (id 1) (at 260.35 98.425 0))
     (property "Footprint" "Diode_SMD:D_SOD-123" (id 2) (at 258.445 95.885 0)
@@
   (symbol (lib_id "Device:R") (at 177.165 100.33 0) (unit 1)
     (in_bom yes) (on_board yes) (fields_autoplaced)
-    (property "Reference" "R17" (id 0) (at 178.943 99.4953 0)
+    (property "Reference" "R16" (id 0) (at 178.943 99.4953 0)
       (effects (font (size 1.27 1.27)) (justify left))
     )
@@
   (symbol (lib_id "Device:D") (at 62.23 95.885 180) (unit 1)
     (in_bom yes) (on_board yes)
-    (property "Reference" "D11" (id 0) (at 62.23 90.1731 0))
+    (property "Reference" "D12" (id 0) (at 62.23 90.1731 0))
     (property "Value" "S1B" (id 1) (at 62.23 92.71 0))
     (property "Footprint" "Diode_SMD:D_SMA" (id 2) (at 62.23 95.885 0)
@@
   (symbol (lib_id "Device:LED") (at 196.85 58.42 90) (unit 1)
     (in_bom yes) (on_board yes)
-    (property "Reference" "D15" (id 0) (at 199.771 59.1728 90)
+    (property "Reference" "D16" (id 0) (at 199.771 59.1728 90)
       (effects (font (size 1.27 1.27)) (justify right))
     )
@@
   (symbol (lib_id "Device:R") (at 119.38 106.045 0) (mirror y) (unit 1)
     (in_bom yes) (on_board yes)
-    (property "Reference" "R16" (id 0) (at 121.9231 106.045 90))
+    (property "Reference" "R15" (id 0) (at 121.9231 106.045 90))
     (property "Value" "10k" (id 1) (at 124.46 106.045 90))
     (property "Footprint" "Resistor_SMD:R_0603_1608Metric" (id 2) (at 121.158 106.045 90)
@@
   (symbol (lib_id "Diode:1N4148") (at 102.87 120.015 180) (unit 1)
     (in_bom yes) (on_board yes) (fields_autoplaced)
-    (property "Reference" "D12" (id 0) (at 102.87 115.0452 0))
+    (property "Reference" "D13" (id 0) (at 102.87 115.0452 0))
     (property "Value" "1N4148" (id 1) (at 102.87 117.5821 0))
     (property "Footprint" "Diode_SMD:D_SOD-123" (id 2) (at 102.87 120.015 0)
@@
   (symbol (lib_id "Device:R") (at 196.85 67.31 0) (unit 1)
     (in_bom yes) (on_board yes) (fields_autoplaced)
-    (property "Reference" "R19" (id 0) (at 198.628 66.4753 0)
+    (property "Reference" "R18" (id 0) (at 198.628 66.4753 0)
       (effects (font (size 1.27 1.27)) (justify left))
     )
@@
   (symbol (lib_id "Device:LED") (at 247.015 100.965 90) (unit 1)
     (in_bom yes) (on_board yes) (fields_autoplaced)
-    (property "Reference" "D16" (id 0) (at 249.936 101.7178 90)
+    (property "Reference" "D17" (id 0) (at 249.936 101.7178 90)
       (effects (font (size 1.27 1.27)) (justify right))
     )
@@
   (symbol (lib_id "Device:R") (at 94.615 65.405 270) (mirror x) (unit 1)
     (in_bom yes) (on_board yes)
-    (property "Reference" "R15" (id 0) (at 94.615 67.9481 90))
+    (property "Reference" "R14" (id 0) (at 94.615 67.9481 90))
     (property "Value" "27" (id 1) (at 94.615 70.485 90))
     (property "Footprint" "Resistor_SMD:R_0603_1608Metric" (id 2) (at 94.615 67.183 90)
@@
   (symbol (lib_id "Device:D_Schottky") (at 122.555 52.705 180) (unit 1)
     (in_bom yes) (on_board yes) (fields_autoplaced)
-    (property "Reference" "D14" (id 0) (at 122.8725 47.7352 0))
+    (property "Reference" "D15" (id 0) (at 122.8725 47.7352 0))
     (property "Value" "RBR1VWM30ATFTR" (id 1) (at 122.8725 50.2721 0))
     (property "Footprint" "Diode_SMD:D_SOD-123" (id 2) (at 122.555 52.705 0)
@@
   (symbol (lib_id "Device:R") (at 177.165 109.22 0) (unit 1)
     (in_bom yes) (on_board yes) (fields_autoplaced)
-    (property "Reference" "R18" (id 0) (at 178.943 108.3853 0)
+    (property "Reference" "R17" (id 0) (at 178.943 108.3853 0)
       (effects (font (size 1.27 1.27)) (justify left))
     )
@@
   (symbol (lib_id "Device:R") (at 216.535 59.69 0) (unit 1)
     (in_bom yes) (on_board yes)
-    (property "Reference" "R20" (id 0) (at 211.455 58.4231 0)
+    (property "Reference" "R19" (id 0) (at 211.455 58.4231 0)
       (effects (font (size 1.27 1.27)) (justify left))
     )
@@
   (symbol (lib_id "Device:R") (at 94.615 62.865 90) (unit 1)
     (in_bom yes) (on_board yes) (fields_autoplaced)
-    (property "Reference" "R14" (id 0) (at 94.615 58.1492 90))
+    (property "Reference" "R13" (id 0) (at 94.615 58.1492 90))
     (property "Value" "27" (id 1) (at 94.615 60.6861 90))
     (property "Footprint" "Resistor_SMD:R_0603_1608Metric" (id 2) (at 94.615 64.643 90)
@@
   (symbol (lib_id "Device:R") (at 247.015 109.855 0) (unit 1)
     (in_bom yes) (on_board yes) (fields_autoplaced)
-    (property "Reference" "R21" (id 0) (at 248.793 109.0203 0)
+    (property "Reference" "R20" (id 0) (at 248.793 109.0203 0)
       (effects (font (size 1.27 1.27)) (justify left))
     )
@@
   (symbol (lib_id "Diode:1N4148") (at 102.87 130.81 180) (unit 1)
     (in_bom yes) (on_board yes) (fields_autoplaced)
-    (property "Reference" "D13" (id 0) (at 102.87 125.8402 0))
+    (property "Reference" "D14" (id 0) (at 102.87 125.8402 0))
     (property "Value" "1N4148" (id 1) (at 102.87 128.3771 0))
     (property "Footprint" "Diode_SMD:D_SOD-123" (id 2) (at 102.87 130.81 0)
@@
   (symbol (lib_id "Diode:1.5KExxA") (at 48.26 101.6 270) (unit 1)
     (in_bom yes) (on_board yes)
-    (property "Reference" "D10" (id 0) (at 50.165 102.235 90)
-      (effects (font (size 1.27 1.27)) (justify left))
-    )
+    (property "Reference" "D11" (id 0) (at 50.165 102.235 90)
+      (effects (font (size 1.27 1.27)) (justify left))
+    )

Commit message: cambiati i pulsanti in smd
se servono gli altri pulsanti usare la versione precedente
Parts:
- SW7: footprint Button_Switch_THT:SW_PUSH_6mm_H5mm -> Button_Switch_SMD:SW_SPST_EVQP0
Changed lines of the file:
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@@
     (property "Reference" "SW7" (id 0) (at 91.44 124.1892 0))
     (property "Value" "Power_button" (id 1) (at 91.44 126.7261 0))
-    (property "Footprint" "Button_Switch_THT:SW_PUSH_6mm_H5mm" (id 2) (at 91.44 125.73 0)
+    (property "Footprint" "Button_Switch_SMD:SW_SPST_EVQP0" (id 2) (at 91.44 125.73 0)
       (effects (font (size 1.27 1.27)) hide)
     )
