File: SCHEMATIC/scheda PSE/scheda PSE.kicad_sch (KiCad schematic)
At the start: 4 parts

Commit message: Aggiunto mosfet uscita corrente usb
Ultima modifica prima della revisone generale.
aggiunto un mosfet P per l'attivazione dell'uscita della tensione alla usb in caso di master
Other:
- sheet Alimentazione ports: added OUTPUT_USB_EN; removed none
- sheet RP2040 ports: added OUTPUT_USB_EN; removed none
Changed lines of the file:
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@@
+    (stroke (width 0) (type default) (color 0 0 0 0))
+  )
+  (wire (pts (xy 114.3 107.95) (xy 68.58 107.95))
     (stroke (width 0) (type default) (color 0 0 0 0))
   )
@@
     (stroke (width 0) (type default) (color 0 0 0 0))
   )
+  (wire (pts (xy 68.58 107.95) (xy 68.58 125.73))
+    (stroke (width 0) (type default) (color 0 0 0 0))
+  )
   (wire (pts (xy 103.505 74.295) (xy 114.3 74.295))
     (stroke (width 0) (type default) (color 0 0 0 0))
@@
   )
   (wire (pts (xy 149.86 87.63) (xy 161.925 87.63))
+    (stroke (width 0) (type default) (color 0 0 0 0))
+  )
+  (wire (pts (xy 68.58 125.73) (xy 74.93 125.73))
     (stroke (width 0) (type default) (color 0 0 0 0))
   )
@@
       (effects (font (size 1.27 1.27)) (justify left))
     )
+    (pin "OUTPUT_USB_EN" input (at 74.93 125.73 180)
+      (effects (font (size 1.27 1.27)) (justify left))
+    )
   )
   (sheet (at 114.3 53.975) (size 35.56 76.835)
@@
     (pin "PWM_SERVO3" output (at 149.86 60.325 0)
       (effects (font (size 1.27 1.27)) (justify right))
+    )
+    (pin "OUTPUT_USB_EN" output (at 114.3 107.95 180)
+      (effects (font (size 1.27 1.27)) (justify left))
     )
   )
@@
       (reference "Q3") (unit 1) (value "IRLML9301") (footprint "Package_TO_SOT_SMD:SOT-23")
     )
+    (path "/7ee2252d-ff7a-4cf9-a8b8-589518dbae10/f4b96b80-f8e2-4d70-bb5d-4a71422936e9"
+      (reference "Q4") (unit 1) (value "IRLML9301") (footprint "Package_TO_SOT_SMD:SOT-23")
+    )
     (path "/788fccce-441b-4b47-abec-e22400b84986/8803450e-3aec-4af4-b3d7-85fb6efd30e4"
       (reference "R1") (unit 1) (value "1k") (footprint "Resistor_SMD:R_0603_1608Metric")
@@
       (reference "R28") (unit 1) (value "470") (footprint "Resistor_SMD:R_0603_1608Metric")
     )
+    (path "/7ee2252d-ff7a-4cf9-a8b8-589518dbae10/62a40344-4203-4e50-bc2b-71e34a2ebebe"
+      (reference "R29") (unit 1) (value "10k") (footprint "Resistor_SMD:R_0603_1608Metric")
+    )
     (path "/9f40c713-1bcb-4f1c-9e01-30533e77b65d/73291c1d-3c5d-4bf2-928d-33312c2dce65"

Commit message: Versione definitiva inviata ai prof
Sistemato tutto e inviato il tutto ai prof
Other:
- sheet RP2040 ports: added none; removed ACC_SA0
- sheet Sensori ports: added none; removed ACC_SA0
Changed lines of the file:
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@@
-    (stroke (width 0) (type default) (color 0 0 0 0))
-  )
-  (wire (pts (xy 149.86 69.215) (xy 161.925 69.215))
     (stroke (width 0) (type default) (color 0 0 0 0))
   )
@@
       (effects (font (size 1.27 1.27)) (justify left))
     )
-    (pin "ACC_SA0" input (at 161.925 69.215 180)
-      (effects (font (size 1.27 1.27)) (justify left))
-    )
     (pin "ESP_TX" output (at 161.925 91.44 180)
       (effects (font (size 1.27 1.27)) (justify left))
@@
     )
     (pin "GPS_PPS" input (at 149.86 85.09 0)
-      (effects (font (size 1.27 1.27)) (justify right))
-    )
-    (pin "ACC_SA0" output (at 149.86 69.215 0)
       (effects (font (size 1.27 1.27)) (justify right))
     )
@@
       (reference "#PWR0105") (unit 1) (value "GND") (footprint "")
     )
+    (path "/7ee2252d-ff7a-4cf9-a8b8-589518dbae10/9e4ac864-2386-4392-9456-227021dbc91f"
+      (reference "#PWR0106") (unit 1) (value "GND") (footprint "")
+    )
+    (path "/7389e30f-cc4a-4964-bca3-cd95052ca62a/f8276108-4e71-4cbf-b8a4-c1496d1ada89"
+      (reference "#PWR0107") (unit 1) (value "GND") (footprint "")
+    )
     (path "/79aec321-3c99-4e59-b384-4589f6950bd0/843d4752-6e63-4d95-a426-482380d37ea8"
       (reference "BZ1") (unit 1) (value "Buzzer") (footprint "_PSE:MLT-8530")
@@
       (reference "R29") (unit 1) (value "10k") (footprint "Resistor_SMD:R_0603_1608Metric")
     )
+    (path "/7ee2252d-ff7a-4cf9-a8b8-589518dbae10/db7ec8b6-f9a8-4b1c-85f3-02bf182afec2"
+      (reference "R30") (unit 1) (value "47k") (footprint "Resistor_SMD:R_0603_1608Metric")
+    )
     (path "/9f40c713-1bcb-4f1c-9e01-30533e77b65d/73291c1d-3c5d-4bf2-928d-33312c2dce65"
